Commit message: scara description and manipulator description. Add separate controllers for manipulator and scara

File: src/manipulator_description/urdf/manipulator/manipulator_ros2_control.urdf.xacro (robot description, xacro)
@@ -5,5 +5,5 @@
     This macro defines the hardware interface for all manipulator joints.
     Uses mock_components/GenericSystem for testing without real hardware.
-    Joints controlled (5 total):
+    Joints controlled (5 base + 3 optional SCARA):
       Main axes (3):
         - base_main_frame_joint (X rail)
@@ -13,6 +13,10 @@
         - selector_left_container_jaw_joint (Y-axis, primary)
         - selector_right_container_jaw_joint (Y-axis, mirrored)
+      SCARA joints (3, optional):
+        - scara_shoulder_joint (Z-axis rotation)
+        - scara_elbow_joint (Z-axis rotation)
+        - scara_wrist_joint (Z-axis rotation)
   -->
-  <xacro:macro name="manipulator_ros2_control">
+  <xacro:macro name="manipulator_ros2_control" params="use_scara:=false">
     <ros2_control name="manipulator_hardware" type="system">
       <!-- Hardware interface plugin -->

File: src/manipulator_description/urdf/robot.urdf.xacro (robot description, xacro)
@@ -21,4 +21,6 @@
   <!-- Load ros2_control hardware interface -->
   <xacro:include filename="$(find manipulator_description)/urdf/manipulator/manipulator_ros2_control.urdf.xacro"/>
+  <!-- Load SCARA ros2_control hardware interface (when SCARA is used) -->
+  <xacro:include filename="$(find scara_description)/urdf/scara_ros2_control.urdf.xacro"/>
   <!-- World link (reference frame) -->
   <link name="world"/>
@@ -35,5 +37,10 @@
   <!-- ros2_control hardware interface (conditional) -->
   <xacro:if value="$(arg use_ros2_control)">
-    <xacro:manipulator_ros2_control/>
+    <xacro:manipulator_ros2_control use_scara="$(arg use_scara)"/>
+    <!-- SCARA ros2_control (only when SCARA is enabled) -->
+    <xacro:if value="$(arg use_scara)">
+      <xacro:scara_ros2_control
+        config_file="$(find scara_description)/config/scara_params.yaml"/>
+    </xacro:if>
   </xacro:if>
 </robot>

File: src/scara_description/urdf/robot.urdf.xacro (robot description, xacro)
@@ -7,7 +7,12 @@
     Usage:
       ros2 launch scara_description display.launch.py
+      ros2 launch scara_description scara_control.launch.py
   -->
+  <!-- Configuration arguments -->
+  <xacro:arg name="use_ros2_control" default="false"/>
   <!-- Include SCARA arm macro -->
   <xacro:include filename="$(find scara_description)/urdf/scara_arm.urdf.xacro"/>
+  <!-- Load ros2_control hardware interface -->
+  <xacro:include filename="$(find scara_description)/urdf/scara_ros2_control.urdf.xacro"/>
   <!-- World link (reference frame) -->
   <link name="world"/>
@@ -45,3 +50,8 @@
     parent_link="base_mount"
     config_file="$(find scara_description)/config/scara_params.yaml"/>
+  <!-- ros2_control hardware interface (conditional) -->
+  <xacro:if value="$(arg use_ros2_control)">
+    <xacro:scara_ros2_control
+      config_file="$(find scara_description)/config/scara_params.yaml"/>
+  </xacro:if>
 </robot>
