Commit message: Добавлены пакет ar4_hardware_interface и прошивка Teensy 4.1. J1+J2+J3+J5 на реальном железе, J4+J6 — mock. J5: NEMA 17 + винт T8. Обновлена документация

File: src/ar4_description/urdf/ar4_ros2_control.urdf.xacro (robot description, xacro)
@@ -3,22 +3,25 @@
   <!--
     ros2_control hardware interface definition for AR4 6-DOF arm
-    Uses mock_components/GenericSystem for testing without real hardware.
-    Joints controlled (6):
-      - J1: Base rotation (Z-axis, ±170°)
-      - J2: Shoulder (Z-axis, -42° to 90°)
-      - J3: Elbow (Z-axis, -89° to 52°)
-      - J4: Wrist roll (Z-axis, ±165°)
-      - J5: Wrist pitch (X-axis, ±105°)
-      - J6: Wrist yaw (Z-axis, ±155°)
+    Two hardware components:
+      1. ar4_real_hardware — real hardware via Teensy 4.1 (J1, J2, J3)
+      2. ar4_mock_hardware — mock for remaining joints (J4-J6)
+    To add a real joint: move its <joint> block from mock to real section
+    and add motor_id, steps_per_rev, gear_ratio, microsteps, home_offset_rad params.
   -->
-  <xacro:macro name="ar4_ros2_control">
-    <ros2_control name="ar4_hardware" type="system">
+  <xacro:macro name="ar4_ros2_control" params="serial_port:=/dev/ttyACM0 baud_rate:=115200">
+    <!-- ============ Real hardware: J1+J2+J3+J5 via Teensy 4.1 ============ -->
+    <ros2_control name="ar4_real_hardware" type="system">
       <hardware>
-        <plugin>mock_components/GenericSystem</plugin>
-        <param name="mock_sensor_commands">true</param>
-        <param name="state_following_offset">0.0</param>
+        <plugin>ar4_hardware_interface/Ar4System</plugin>
+        <param name="serial_port">${serial_port}</param>
+        <param name="baud_rate">${baud_rate}</param>
       </hardware>
       <!-- J1: Base rotation -->
       <joint name="J1">
+        <param name="motor_id">0</param>
+        <param name="steps_per_rev">200</param>
+        <param name="gear_ratio">40.0</param>
+        <param name="microsteps">16</param>
+        <param name="home_offset_rad">2.967</param>
         <command_interface name="position">
           <param name="min">${radians(-170)}</param>
@@ -32,6 +35,11 @@
       <!-- J2: Shoulder -->
       <joint name="J2">
+        <param name="motor_id">1</param>
+        <param name="steps_per_rev">200</param>
+        <param name="gear_ratio">40.0</param>
+        <param name="microsteps">16</param>
+        <param name="home_offset_rad">-0.7330</param>
         <command_interface name="position">
-          <param name="min">${radians(-42)}</param>
+          <param name="min">${radians(-44)}</param>
           <param name="max">${radians(90)}</param>
         </command_interface>
@@ -43,4 +51,9 @@
       <!-- J3: Elbow -->
       <joint name="J3">
+        <param name="motor_id">2</param>
+        <param name="steps_per_rev">200</param>
+        <param name="gear_ratio">50.0</param>
+        <param name="microsteps">16</param>
+        <param name="home_offset_rad">-1.5533</param>
         <command_interface name="position">
           <param name="min">${radians(-89)}</param>
@@ -52,9 +65,15 @@
         <state_interface name="velocity"/>
       </joint>
-      <!-- J4: Wrist roll -->
-      <joint name="J4">
+      <!-- J5: Wrist pitch — NEMA 17 + MKS SERVO42C + T8 lead screw (no gear reducer)
+           PLACEHOLDER gear_ratio — calibrate empirically with real hardware -->
+      <joint name="J5">
+        <param name="motor_id">3</param>
+        <param name="steps_per_rev">200</param>
+        <param name="gear_ratio">1.0</param>
+        <param name="microsteps">16</param>
+        <param name="home_offset_rad">1.7104</param>
         <command_interface name="position">
-          <param name="min">${radians(-165)}</param>
-          <param name="max">${radians(165)}</param>
+          <param name="min">${radians(-105)}</param>
+          <param name="max">${radians(105)}</param>
         </command_interface>
         <state_interface name="position">
@@ -63,9 +82,17 @@
         <state_interface name="velocity"/>
       </joint>
-      <!-- J5: Wrist pitch -->
-      <joint name="J5">
+    </ros2_control>
+    <!-- ============ Mock hardware: J4+J6 ============ -->
+    <ros2_control name="ar4_mock_hardware" type="system">
+      <hardware>
+        <plugin>mock_components/GenericSystem</plugin>
+        <param name="mock_sensor_commands">true</param>
+        <param name="state_following_offset">0.0</param>
+      </hardware>
+      <!-- J4: Wrist roll -->
+      <joint name="J4">
         <command_interface name="position">
-          <param name="min">${radians(-105)}</param>
-          <param name="max">${radians(105)}</param>
+          <param name="min">${radians(-165)}</param>
+          <param name="max">${radians(165)}</param>
         </command_interface>
         <state_interface name="position">

File: src/ar4_description/urdf/robot.urdf.xacro (robot description, xacro)
@@ -10,4 +10,6 @@
   <!-- Arguments -->
   <xacro:arg name="use_ros2_control" default="true"/>
+  <xacro:arg name="serial_port" default="/dev/ttyACM0"/>
+  <xacro:arg name="baud_rate" default="115200"/>
   <!-- Include macros -->
   <xacro:include filename="$(find ar4_description)/urdf/ar4_macro.xacro"/>
@@ -21,5 +23,5 @@
   <!-- ros2_control hardware interface -->
   <xacro:if value="$(arg use_ros2_control)">
-    <xacro:ar4_ros2_control/>
+    <xacro:ar4_ros2_control serial_port="$(arg serial_port)" baud_rate="$(arg baud_rate)"/>
   </xacro:if>
 </robot>

Commit message: Добавлены J4 и J6 в прошивку и URDF, перенумерован J5. NUM_JOINTS=6, все суставы на реальном железе. J4: NEMA 11 + 40:1 (STEP=6, DIR=7, LIMIT=26). J6: NEMA 14 +   MKS 35D RS485 + 19:1 (STEP=10, DIR=11, LIMIT=28). Удалена mock-секция из URDF. Обновлена документация.

File: src/ar4_description/urdf/ar4_ros2_control.urdf.xacro (robot description, xacro)
@@ -3,12 +3,8 @@
   <!--
     ros2_control hardware interface definition for AR4 6-DOF arm
-    Two hardware components:
-      1. ar4_real_hardware — real hardware via Teensy 4.1 (J1, J2, J3)
-      2. ar4_mock_hardware — mock for remaining joints (J4-J6)
-    To add a real joint: move its <joint> block from mock to real section
-    and add motor_id, steps_per_rev, gear_ratio, microsteps, home_offset_rad params.
+    All 6 joints driven by real hardware via Teensy 4.1.
   -->
   <xacro:macro name="ar4_ros2_control" params="serial_port:=/dev/ttyACM0 baud_rate:=115200">
-    <!-- ============ Real hardware: J1+J2+J3+J5 via Teensy 4.1 ============ -->
+    <!-- ============ Real hardware: J1–J6 via Teensy 4.1 ============ -->
     <ros2_control name="ar4_real_hardware" type="system">
       <hardware>
@@ -65,8 +61,24 @@
         <state_interface name="velocity"/>
       </joint>
+      <!-- J4: Wrist roll — NEMA 11 + MKS SERVO42C + 40:1 planetary -->
+      <joint name="J4">
+        <param name="motor_id">3</param>
+        <param name="steps_per_rev">200</param>
+        <param name="gear_ratio">40.0</param>
+        <param name="microsteps">16</param>
+        <param name="home_offset_rad">-3.1416</param>
+        <command_interface name="position">
+          <param name="min">${radians(-165)}</param>
+          <param name="max">${radians(165)}</param>
+        </command_interface>
+        <state_interface name="position">
+          <param name="initial_value">0.0</param>
+        </state_interface>
+        <state_interface name="velocity"/>
+      </joint>
       <!-- J5: Wrist pitch — NEMA 17 + MKS SERVO42C + T8 lead screw (no gear reducer)
            PLACEHOLDER gear_ratio — calibrate empirically with real hardware -->
       <joint name="J5">
-        <param name="motor_id">3</param>
+        <param name="motor_id">4</param>
         <param name="steps_per_rev">200</param>
         <param name="gear_ratio">1.0</param>
@@ -82,25 +94,11 @@
         <state_interface name="velocity"/>
       </joint>
-    </ros2_control>
-    <!-- ============ Mock hardware: J4+J6 ============ -->
-    <ros2_control name="ar4_mock_hardware" type="system">
-      <hardware>
-        <plugin>mock_components/GenericSystem</plugin>
-        <param name="mock_sensor_commands">true</param>
-        <param name="state_following_offset">0.0</param>
-      </hardware>
-      <!-- J4: Wrist roll -->
-      <joint name="J4">
-        <command_interface name="position">
-          <param name="min">${radians(-165)}</param>
-          <param name="max">${radians(165)}</param>
-        </command_interface>
-        <state_interface name="position">
-          <param name="initial_value">0.0</param>
-        </state_interface>
-        <state_interface name="velocity"/>
-      </joint>
-      <!-- J6: Wrist yaw -->
+      <!-- J6: Wrist yaw — NEMA 14 + MKS 35D RS485 + 19:1 built-in planetary -->
       <joint name="J6">
+        <param name="motor_id">5</param>
+        <param name="steps_per_rev">200</param>
+        <param name="gear_ratio">19.0</param>
+        <param name="microsteps">16</param>
+        <param name="home_offset_rad">3.1416</param>
         <command_interface name="position">
           <param name="min">${radians(-155)}</param>
